File: CMOY.sch (KiCad schematic (older format))
At the start: 18 parts, among them IC1 OPA2134P, U1 NMA0512SC

Commit message: Updated Design Files
Parts:
- added C19: C, Capacitors_SMD:C_0805_HandSoldering, symbol Device:C
- added L2: L, Capacitors_SMD:C_0805_HandSoldering, symbol Device:L
- added unit 1 of M1
- C1, C6: symbol CAPACITOR-WIMA_C5_5 -> USBDACCMOY-rescue:CAPACITOR-WIMA_C5_5
- C2, C4: symbol RCL_CPOL-USE3.5-8 -> USBDACCMOY-rescue:RCL_CPOL-USE3.5-8
- C3, C5: symbol CAPACITOR-WIMA_C2.5_2 -> USBDACCMOY-rescue:CAPACITOR-WIMA_C2.5_2
- IC1: footprint CMOY:DIL-8 -> SMD_Packages:SOIC-8-N; symbol OPA2134P -> USBDACCMOY-rescue:OPA2134P
- JACK-OUT1: symbol STEREOJACK -> USBDACCMOY-rescue:STEREOJACK
- M1: renamed from U$1; value ~ -> AUDIO-POTS_ALPS_RK0971221Z05; footprint CMOY:AUDIO-POTS_ALPS_RK0971221Z0X -> PCM2707:AUDIO-POTS_ALPS_RK0971221Z0X; symbol AUDIO-POTS_ALPS_RK0971221Z05 -> USBDACCMOY-rescue:AUDIO-POTS_ALPS_RK0971221Z05
- R1, R2, R3, R4, R5, R6, R7, R8: symbol RESISTOR_R-EU_0207_2V -> USBDACCMOY-rescue:RESISTOR_R-EU_0207_2V
- U1: symbol NMA0512SC -> USBDACCMOY-rescue:NMA0512SC
Connections:
- net labels added: GND
- net labels removed: AESTHETICS_GND
- wire segments 55 -> 74
