File: PCM2707.sch (KiCad schematic (older format))
At the start: 36 parts, among them CON1 GND_CONNECTORSMD, J1 USB, Q1 12MHz, U2 PCM2707C

Commit message: Updated Design Files
Parts:
- C10, C9: symbol CAP1210 -> USBDACCMOY-rescue:CAP1210
- C11, C12, C14, C15, C16, C17, C18: symbol CAP0805 -> USBDACCMOY-rescue:CAP0805
- C13: symbol CAP_POLC -> USBDACCMOY-rescue:CAP_POLC
- C7, C8: symbol CAP_POLD -> USBDACCMOY-rescue:CAP_POLD
- CON1: symbol GND_CONNECTORSMD -> USBDACCMOY-rescue:GND_CONNECTORSMD
- DOUT1: symbol CON-MOLEX_87758-0216 -> USBDACCMOY-rescue:CON-MOLEX_87758-0216
- J1: symbol MOLEX-47346-0001_47346-0001 -> USBDACCMOY-rescue:MOLEX-47346-0001_47346-0001
- JP1: symbol CONNECTORS_M05LOCK -> USBDACCMOY-rescue:CONNECTORS_M05LOCK
- L1: symbol INDUCTOR0805 -> USBDACCMOY-rescue:INDUCTOR0805
- LED1, LED2: symbol LED_LED0603 -> USBDACCMOY-rescue:LED_LED0603
- OUTPUT1: symbol CON-LSTB_MA03-1 -> USBDACCMOY-rescue:CON-LSTB_MA03-1
- Q1: symbol CRYSTAL_CRYSTALHC49U-V -> USBDACCMOY-rescue:CRYSTAL_CRYSTALHC49U-V
- R10, R11, R12, R13, R14, R15, R16, R17, R18, R19, R20, R21, R9: symbol RESISTOR0805-RES -> USBDACCMOY-rescue:RESISTOR0805-RES
- SV1: symbol CON-LSTB_MA04-1 -> USBDACCMOY-rescue:CON-LSTB_MA04-1
- U2: symbol PCM2707C -> USBDACCMOY-rescue:PCM2707C
Connections:
- net VBUS: no longer C15.1, L1.1, U2.24 (VBUS)
- new net: C15.1, L1.1, U2.24 (VBUS)
